File: mcu_board_1.kicad_pcb (KiCad board)
At the start: 2 copper layers, 125 parts, among them J1 Conn_01x03, J10 Conn_01x03, J11 USB-B_WE_61400416121, J12 Conn_01x03, J13 Conn_01x02, J14 Conn_01x08, J15 Conn_01x03, J16 +15V, J17 GND, J18 WE 691216710002, J19 Conn_02x04_Counter_Clockwise, J2 ARM_SWD_10, J20 Conn_02x04_Counter_Clockwise, J21 Conn_02x04_Counter_Clockwise, J3 Conn_02x20_Top_Bottom, J4 Conn_02x20_Top_Bottom, J5 Conn_02x12_Top_Bottom, J6 Conn_01x02, J7 Conn_02x04_Top_Bottom, J8 Conn_02x03_Top_Bottom, J9 Conn_01x06, Q1 2N7002BK,215, Q2 2N7002BK,215, Q3 2N7002BK,215, SW1 SW_SPST, SW2 Rotary_Encoder_Switch, SW3 SW_SPST, SW4 SW_SPST, SW5 SW_SPST, U1 STM32G474QET6, U2 REF5040, U3 OPA333AID, U4 50k 0.1%, U5 OPA333AID, U6 FT232RL, U7 M95M01-R, U8 AMS1117-3.3, U9 AMS1117-3.3, Y1 32.7680kHz, Y2 10MHz

Commit message: MCU prepped for fanout
Parts:
- J19, J20, J21: value Conn_02x04_Counter_Clockwise -> Conn_02x04_Odd_Even
- J3, J4: value Conn_02x20_Top_Bottom -> Conn_02x20_Odd_Even
- J5: value Conn_02x12_Top_Bottom -> Conn_02x12_Odd_Even
- J7: value Conn_02x04_Top_Bottom -> Conn_02x04_Odd_Even
- J8: value Conn_02x03_Top_Bottom -> Conn_02x03_Odd_Even
- moved D5 319.1 mm to (247.8, -51.2)
- moved D3 317.6 mm to (247.8, -70.8)
- moved D4 311.7 mm to (247.8, -61.0)
- moved R6 308.9 mm to (256.6, -118.4)
- moved R5 262.8 mm to (253.4, -118.3)
- moved R11 262.8 mm to (255.4, -112.9)
- moved R10 254.8 mm to (250.9, -113.2)
- moved R9 254.3 mm to (254.7, -115.6)
- moved C22 252.4 mm to (250.6, -128.2)
- moved U7 249.2 mm to (253.4, -124.0)
- moved R8 247.9 mm to (251.0, -116.1)
- moved SW4 243.6 mm to (234.4, -53.6)
- moved D2 228.0 mm to (138.1, -99.4), turned to 90 degrees
- moved KB1 224.3 mm to (175.0, -73.0)
- moved SW5 223.6 mm to (234.4, -63.3)
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Connections:
- J19 pad 2: +15V -> GND
- J19 pad 4: +15V -> GND
- J19 pad 5: GND -> +15V
- J19 pad 7: GND -> +15V
- J20 pad 2: +5V -> GND
- J20 pad 4: +5V -> GND
- J20 pad 5: GND -> +5V
- J20 pad 7: GND -> +5V
- J21 pad 2: +3V3 -> GND
- J21 pad 4: +3V3 -> GND
- J21 pad 5: GND -> +3V3
- J21 pad 7: GND -> +3V3
- J3 pad 1: PE2 -> PE8
- J3 pad 10: PF7 -> PB0
- J3 pad 11: PF8 -> PC5
- J3 pad 12: PF9 -> PC4
- J3 pad 13: PF10 -> PA7
- J3 pad 14: PG10 -> PA6
- J3 pad 15: PC0 -> PA5
- J3 pad 16: PC1 -> PA4
- J3 pad 17: PC2 -> PA3
- J3 pad 18: PC3 -> PA2
- J3 pad 19: PF2 -> PA1
- J3 pad 2: PE3 -> PE7
- J3 pad 21: PB10 -> PF2
- J3 pad 22: PE15 -> PC3
- J3 pad 23: PE14 -> PC2
- J3 pad 24: PE13 -> PC1
- J3 pad 25: PE12 -> PC0
- J3 pad 26: PE11 -> PG10
- J3 pad 27: PE10 -> PF10
- J3 pad 28: PE9 -> PF9
- J3 pad 29: PE8 -> PF8
- J3 pad 3: PE4 -> PF15
- J3 pad 30: PE7 -> PF7
- J3 pad 31: PF15 -> PF5
- J3 pad 32: PF14 -> PF4
- J3 pad 33: PF13 -> PF3
- J3 pad 34: PF12 -> PC13
- J3 pad 35: PF11 -> PE6
- J3 pad 36: PD7 -> PE5
- J3 pad 37: PB3 -> PE4
- J3 pad 38: PB4 -> PE3
- J3 pad 39: PB5 -> PE2
- J3 pad 4: PE5 -> PF14
- J3 pad 40: PB6 -> GND
- J3 pad 5: PE6 -> PF13
- J3 pad 6: PC13 -> PF12
- J3 pad 7: PF3 -> PF11
- J3 pad 8: PF4 -> PB2
- J3 pad 9: PF5 -> PB1
- J4 pad 1: PA1 -> PC10
- J4 pad 10: PG5 -> PA8
- J4 pad 11: PG6 -> PC9
- J4 pad 12: PG7 -> PC8
- J4 pad 13: PG8 -> PG4
- J4 pad 14: PG9 -> PG3
- J4 pad 15: PD0 -> PG2
- J4 pad 16: PD1 -> PG1
- J4 pad 17: PD2 -> PG0
- J4 pad 18: PD3 -> PC7
- J4 pad 19: PD4 -> PC6
- J4 pad 2: PA2 -> PA15
- J4 pad 20: PD5 -> PD15
- J4 pad 21: PB2 -> PD14
- J4 pad 22: PB1 -> PD13
- J4 pad 23: PB0 -> PD12
- J4 pad 24: PC5 -> PD11
- J4 pad 25: PC4 -> PD10
- J4 pad 26: PA7 -> PD9
- J4 pad 27: PA6 -> PD8
- J4 pad 28: PA5 -> PB15
- J4 pad 29: PA4 -> PB14
- J4 pad 3: PA3 -> PA14
- J4 pad 30: PB7 -> PB13
- J4 pad 31: PB8 -> PB12
- J4 pad 32: PB9 -> PB11
- J4 pad 33: PE0 -> PB10
- J4 pad 34: PE1 -> PE15
- J4 pad 35: PD6 -> PE14
- J4 pad 36: PB15 -> PE13
- J4 pad 37: PB14 -> PE12
- J4 pad 38: PB13 -> PE11
- J4 pad 39: PB12 -> PE10
- J4 pad 40: PB11 -> PE9
- J4 pad 5: PA14 -> PA13
- J4 pad 6: PA15 -> PA12
- J4 pad 7: PC10 -> PA11
- J4 pad 8: PC11 -> PA10
- J4 pad 9: PC12 -> PA9
- J5 pad 1: PG0 -> PE1
- J5 pad 10: PD9 -> PD7
- J5 pad 11: PD8 -> PD6
- J5 pad 12: GND -> PD5
- J5 pad 13: PA13 -> PD4
- J5 pad 14: PA12 -> PD3
- J5 pad 15: PA11 -> PD2
- J5 pad 16: PA10 -> PD1
- J5 pad 17: PA9 -> PD0
- J5 pad 18: PA8 -> PG9
- J5 pad 19: PC9 -> PG8
- J5 pad 2: PC7 -> PE0
- J5 pad 20: PC8 -> PG7
- J5 pad 21: PG4 -> PG6
- J5 pad 22: PG3 -> PG5
- J5 pad 23: PG2 -> PC12
- J5 pad 24: PG1 -> PC11
- J5 pad 3: PC6 -> PB9
- J5 pad 4: PD15 -> PB8
- J5 pad 5: PD14 -> PB7
- J5 pad 6: PD13 -> PB6
- J5 pad 7: PD12 -> PB5
- J5 pad 8: PD11 -> PB4
- J5 pad 9: PD10 -> PB3
- J7 pad 2: /Analog/3_4_REF -> Net-(J7-Pad2)
- J7 pad 3: /Analog/2_4_REF -> /Analog/3_4_REF
- J7 pad 4: /Analog/1_4_REF -> Net-(J7-Pad2)
- J7 pad 5: Net-(J7-Pad5) -> /Analog/2_4_REF
- J7 pad 6: Net-(J7-Pad5) -> Net-(J7-Pad2)
- J7 pad 7: Net-(J7-Pad5) -> /Analog/1_4_REF
- J7 pad 8: Net-(J7-Pad5) -> Net-(J7-Pad2)
- J8 pad 2: GND -> /REF
- J8 pad 5: /REF -> GND
- U5 pad 3: Net-(J7-Pad5) -> Net-(J7-Pad2)
Other:
- board text added: "0.25"
- board text added: "0.50"
- board text added: "0.75"
- board text added: "1.00"
- board text added: "BUT 1"
- board text added: "BUT 2"
- board text added: "BUT 3"
- board text added: "LED 1"
- board text added: "LED 2"
- board text added: "LED 3"

Commit message: done and done
Parts:
- added C36: 100n, Capacitor_SMD:C_0603_1608Metric_Pad1.05x0.95mm_HandSolder, F.Cu at (154.3, 102.0)
- added C37: 1U, Capacitor_SMD:C_0603_1608Metric_Pad1.05x0.95mm_HandSolder, F.Cu at (180.7, 79.5)
- added H1: MountingHole_Pad, MountingHole:MountingHole_3.2mm_M3_Pad_Via, F.Cu at (220.0, 22.5)
- added H2: MountingHole_Pad, MountingHole:MountingHole_3.2mm_M3_Pad_Via, F.Cu at (220.0, 147.5)
- added H3: MountingHole_Pad, MountingHole:MountingHole_3.2mm_M3_Pad_Via, F.Cu at (80.0, 22.5)
- added H4: MountingHole_Pad, MountingHole:MountingHole_3.2mm_M3_Pad_Via, F.Cu at (80.0, 147.5)
- added R38: DNP, Resistor_SMD:R_0603_1608Metric_Pad1.05x0.95mm_HandSolder, F.Cu at (175.1, 47.4)
- added R39: 47k 1%, Resistor_SMD:R_0603_1608Metric_Pad1.05x0.95mm_HandSolder, F.Cu at (175.1, 43.6)
- moved R4 276.1 mm to (204.2, 131.6), turned to 90 degrees
- moved J10 272.5 mm to (206.7, 128.3), turned to 270 degrees
- moved R19 271.5 mm to (187.1, 144.3), turned to 270 degrees
- moved R3 269.4 mm to (206.7, 131.6), turned to 90 degrees
- moved J2 268.8 mm to (214.0, 37.2), turned to 180 degrees
- moved R7 266.6 mm to (201.6, 131.6), turned to 90 degrees
- moved J14 266.5 mm to (125.0, 147.5), turned to 270 degrees
- moved R31 261.8 mm to (153.9, 141.6), turned to 90 degrees
- moved C15 261.5 mm to (211.0, 42.8), turned to 270 degrees
- moved R18 261.4 mm to (177.3, 144.3), turned to 270 degrees
- moved J12 260.8 mm to (187.9, 129.5), turned to 90 degrees
- moved R16 260.3 mm to (188.0, 132.7), turned to 90 degrees
- moved Q3 260.1 mm to (157.6, 137.0), turned to 270 degrees
- moved R17 259.5 mm to (167.6, 144.3), turned to 270 degrees
- moved R12 257.7 mm to (193.0, 132.6), turned to 90 degrees
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Connections:
- C6 pad 1: GNDA -> GND
- J1 pad 2: GND -> Net-(C5-Pad2)
- J1 pad 3: Net-(C5-Pad2) -> GND
- U1 pad 42: GNDA -> GND
Routing:
- net GND: track 0.00 -> 1125.2 mm, vias 0 -> 23
- net +3V3: track 0.00 -> 449.8 mm, vias 0 -> 23
- net +5V: track 0.00 -> 220.6 mm, vias 0 -> 5
- net +3.3VA: track 0.00 -> 196.9 mm, vias 0 -> 6
- net PG10: track 0.00 -> 146.2 mm, vias 0 -> 2
- net /REF: track 0.00 -> 133.0 mm, vias 0 -> 2
- net PE3: track 0.00 -> 73.0 mm
- net PE2: track 0.00 -> 71.1 mm
- net +15V: track 0.00 -> 71.0 mm
- net PE5: track 0.00 -> 70.9 mm
- net PE4: track 0.00 -> 68.8 mm
- net PE6: track 0.00 -> 66.9 mm
- net PC13: track 0.00 -> 62.4 mm, vias 0 -> 2
- net PF4: track 0.00 -> 61.4 mm, vias 0 -> 2
- net PB3: track 0.00 -> 60.8 mm
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- added copper zone on B.Cu, net GND
- added copper zone on F.Cu, net GND
Other:
- board outline added: 150 x 135 mm
- net class Default: clearance 0.2 -> 0.15; trace_width 0.25 -> 0.2
- rule trace_clearance: 0.2 -> 0.15
- board text added: "09.11.2020"
- board text added: "15V"
- board text added: "3V3"
- board text added: "3V3A"
- board text added: "5V"
- board text added: "A"
- board text added: "B"
- board text added: "BAT"
- board text added: "BUT1"
- board text added: "BUT2"
- board text added: "BUT3"
- board text added: "C"
- board text added: "C1"
- board text added: "C2"
- board text added: "C3"
- board text added: "C4"
- board text added: "COM"
- board text added: "D"
- board text added: "EEPROM"
- board text added: "G"
- board text added: "GND"
- board text added: "HT Blog"
- board text added: "LED1"
- board text added: "LED2"
- board text added: "LED3"
- board text added: "PA0"
- board text added: "PA1"
- board text added: "PA10"
- board text added: "PA11"
- board text added: "PA12"
- board text added: "PA13"
- board text added: "PA14"
- board text added: "PA15"
- board text added: "PA2"
- board text added: "PA3"
- board text added: "PA4"
- board text added: "PA5"
- board text added: "PA6"
- board text added: "PA7"
- board text added: "PA8"
- board text added: "PA9"
- board text added: "PB0"
- board text added: "PB1"
- board text added: "PB10"
- board text added: "PB11"
- board text added: "PB12"
- board text added: "PB13"
- board text added: "PB14"
- board text added: "PB15"
- board text added: "PB2"
- board text added: "PB3"
- board text added: "PB4"
- board text added: "PB5"
- board text added: "PB6"
- board text added: "PB7"
- board text added: "PB8"
- board text added: "PB9"
- board text added: "PC0"
- board text added: "PC1"
- board text added: "PC10"
- board text added: "PC11"
- board text added: "PC12"
- board text added: "PC13"
- board text added: "PC2"
- board text added: "PC3"
- board text added: "PC4"
- board text added: "PC5"
- board text added: "PC6"
- board text added: "PC7"
- board text added: "PC8"
- board text added: "PC9"
- board text added: "PD0"
- board text added: "PD1"
- board text added: "PD10"
- board text added: "PD11"
- board text added: "PD12"
- board text added: "PD13"
- board text added: "PD14"
- board text added: "PD15"
- board text added: "PD2"
- board text added: "PD3"
- board text added: "PD4"
- board text added: "PD5"
- board text added: "PD6"
- board text added: "PD7"
- board text added: "PD8"
- board text added: "PD9"
- board text added: "PE0"
- board text added: "PE1"
- board text added: "PE10"
- board text added: "PE11"
- board text added: "PE12"
- board text added: "PE13"
- board text added: "PE14"
- board text added: "PE15"
- board text added: "PE2"
- board text added: "PE3"
- board text added: "PE4"
- board text added: "PE5"
- board text added: "PE6"
- board text added: "PE7"
- board text added: "PE8"
- board text added: "PE9"
- board text added: "PF10"
- board text added: "PF11"
- board text added: "PF12"
- board text added: "PF13"
- board text added: "PF14"
- board text added: "PF15"
- board text added: "PF2"
- board text added: "PF3"
- board text added: "PF4"
- board text added: "PF5"
- board text added: "PF6"
- board text added: "PF7"
- board text added: "PF8"
- board text added: "PF9"
- board text added: "PG0"
- board text added: "PG1"
- board text added: "PG10"
- board text added: "PG2"
- board text added: "PG3"
- board text added: "PG4"
- board text added: "PG5"
- board text added: "PG6"
- board text added: "PG7"
- board text added: "PG8"
- board text added: "PG9"
- board text added: "Q"
- board text added: "R1"
- board text added: "R2"
- board text added: "R3"
- board text added: "R4"
- board text added: "REF"
- board text added: "REF SET"
- board text added: "RESET"
- board text added: "RX"
- board text added: "SMU MCU BOARD"
- board text added: "STM32G474QET6"
- board text added: "SW"
- board text added: "SWD"
- board text added: "T"
- board text added: "TX"
- board text added: "V.1"
- board text added: "~HOLD"
- board text added: "~S"
- board text added: "~W"
